Commit message: Increase simulation navigation speed and lidar update rate

File: ros_ws/src/my_bot/description/simulation_parameters.xacro (robot description, xacro)
@@ -14,5 +14,5 @@
   <xacro:property name="wheel_friction" value="0.8"/>
   <xacro:property name="caster_friction" value="0.001"/>
-  <xacro:property name="scan_hz" value="10"/>
+  <xacro:property name="scan_hz" value="15"/>
   <xacro:property name="scan_samples" value="360"/>
   <xacro:property name="scan_min" value="0.15"/>
